Commit message: solve the lidar frame problem which caused the lidar visualization problem in rviz

File: src/tow_tractor_description/urdf/tow_tractor_v1/gazebo_lidar.xacro (robot description, xacro)
@@ -31,5 +31,6 @@
     </joint>
     <gazebo reference="lidar_frame">
-        <sensor name='lidar_sensor' type='gpu_lidar'>
+        <sensor name='lidar_frame' type='gpu_lidar'>
+            <gz_frame_id>lidar_frame</gz_frame_id>
             <always_on>true</always_on>
             <visualize>true</visualize>

File: src/tow_tractor_description/urdf/tow_tractor_v1/tow_tractor_v1_core.xacro (robot description, xacro)
@@ -22,4 +22,12 @@
     <link name="base_link">
     </link>
+    <!-- BASE FOOTPRINT LINK -->
+    <link name ="base_footprint">
+    </link>
+    <joint name="base_footprint_joint" type="fixed">
+        <parent link="base_link"/>
+        <child link="base_footprint"/>
+        <origin xyz="0 0.0 0.0" rpy="0.0 0.0 0.0"/>
+    </joint>
     <!-- CHASSIS LINK -->
     <link name="chassis_link">
