Commit message: created odom_pub_node to calc odom and joint_states unfiltered, imu_frame to imu received msg and added time stamped to imu received msgs, isolated the links from gazebo plugins to the normal urdf, added odom to launch file

File: src/tow_tractor_description/urdf/tow_tractor_v2/gazebo_imu.xacro (robot description, xacro)
@@ -1,12 +1,4 @@
 <?xml version="1.0"?>
 <robot xmlns:xacro="http://www.ros.org/wiki/xacro">
-    <!-- LIDAR LINK -->
-    <link name="imu_frame">
-    </link>
-    <joint name="imu_joint" type="fixed">
-        <parent link="chassis_link"/>
-        <child link="imu_frame"/>
-        <origin xyz="${chassis_width / 2} 0.0 ${chassis_hight / 2}" rpy="0.0 0.0 0.0"/>
-    </joint>
     <gazebo reference="imu_frame">
         <sensor name="imu_sensor" type="imu">

File: src/tow_tractor_description/urdf/tow_tractor_v2/gazebo_lidar.xacro (robot description, xacro)
@@ -1,33 +1,4 @@
 <?xml version="1.0"?>
 <robot xmlns:xacro="http://www.ros.org/wiki/xacro">
-    <!-- SENSORS -->
-    <xacro:property name="lidar_rad" value="0.038"/>
-    <xacro:property name="lidar_width" value="0.0335"/>
-    <xacro:property name="lidar_material" value="black"/>
-    <xacro:property name="lidar_mass" value="0.042"/>
-    <!-- LIDAR LINK -->
-    <link name="lidar_frame">
-        <visual>
-            <geometry>
-                <cylinder radius="${lidar_rad}" length="${lidar_width}"/>
-            </geometry>
-            <origin xyz="0.0 0.0 0" rpy="0.0 0.0 0.0"/>
-            <material name="${lidar_material}"/>
-        </visual>
-        <collision>
-            <geometry>
-                <cylinder radius="${lidar_rad}" length="${lidar_width}"/>
-            </geometry>
-            <origin xyz="0.0 0.0 ${chassis_hight + lidar_width / 2}" rpy="0.0 0.0 0.0"/>
-        </collision>
-        <xacro:inertial_cylinder mass="${lidar_mass}" radius="${lidar_rad}" length="${lidar_width}">
-            <origin xyz="0.0 0.0 0.0" rpy="0.0 0.0 0.0"/>
-        </xacro:inertial_cylinder>
-    </link>
-    <joint name="lidar_joint" type="fixed">
-        <parent link="base_link"/>
-        <child link="lidar_frame"/>
-        <origin xyz="0.0 0.0 ${chassis_hight + lidar_width / 2}" rpy="0.0 0.0 0.0"/>
-    </joint>
     <gazebo reference="lidar_frame">
         <sensor name='lidar_frame' type='gpu_lidar'>

File: src/tow_tractor_description/urdf/tow_tractor_v2/tow_tractor_v2_core.xacro (robot description, xacro)
@@ -19,4 +19,9 @@
     <xacro:property name="steering_max_speed" value="1.0"/>         <!--rad/s-->
     <xacro:property name="steering_max_torque" value="10.0"/>       <!-- N.m-->
+    <!-- SENSORS -->
+    <xacro:property name="lidar_rad" value="0.038"/>
+    <xacro:property name="lidar_width" value="0.0335"/>
+    <xacro:property name="lidar_material" value="black"/>
+    <xacro:property name="lidar_mass" value="0.042"/>
     <!-- BASE LINK -->
     <link name="base_link">
@@ -156,3 +161,35 @@
         <mu2 value="0.001"/>
     </gazebo>
+    <!-- IMU LINK -->
+    <link name="imu_frame">
+    </link>
+    <joint name="imu_joint" type="fixed">
+        <parent link="chassis_link"/>
+        <child link="imu_frame"/>
+        <origin xyz="${chassis_width / 2} 0.0 ${chassis_hight / 2}" rpy="0.0 0.0 0.0"/>
+    </joint>
+    <!-- LIDAR LINK -->
+    <link name="lidar_frame">
+        <visual>
+            <geometry>
+                <cylinder radius="${lidar_rad}" length="${lidar_width}"/>
+            </geometry>
+            <origin xyz="0.0 0.0 0" rpy="0.0 0.0 0.0"/>
+            <material name="${lidar_material}"/>
+        </visual>
+        <collision>
+            <geometry>
+                <cylinder radius="${lidar_rad}" length="${lidar_width}"/>
+            </geometry>
+            <origin xyz="0.0 0.0 ${chassis_hight + lidar_width / 2}" rpy="0.0 0.0 0.0"/>
+        </collision>
+        <xacro:inertial_cylinder mass="${lidar_mass}" radius="${lidar_rad}" length="${lidar_width}">
+            <origin xyz="0.0 0.0 0.0" rpy="0.0 0.0 0.0"/>
+        </xacro:inertial_cylinder>
+    </link>
+    <joint name="lidar_joint" type="fixed">
+        <parent link="base_link"/>
+        <child link="lidar_frame"/>
+        <origin xyz="0.0 0.0 ${chassis_hight + lidar_width / 2}" rpy="0.0 0.0 0.0"/>
+    </joint>
 </robot>
