Commit message: added lidar stl file to the robot description, configured and added lidar driver, added navigation package, (needs tunning)

File: src/tow_tractor_description/urdf/tow_tractor_v2/tow_tractor_v2_core.xacro (robot description, xacro)
@@ -170,11 +170,13 @@
     </joint>
     <!-- LIDAR LINK -->
-    <link name="lidar_frame">
-        <visual>
-            <geometry>
-                <cylinder radius="${lidar_rad}" length="${lidar_width}"/>
-            </geometry>
-            <origin xyz="0.0 0.0 0" rpy="0.0 0.0 0.0"/>
-            <material name="${lidar_material}"/>
+    <link name="lidar_base">
+        <visual>
+            <origin xyz="0 0 0" rpy="0 0 0"/>
+            <geometry>
+                <mesh filename="package://tow_tractor_description/meshes/LD19.stl" scale="0.001 0.001 0.001" />
+            </geometry>
+            <material name="ldlidar_mat">
+                <color rgba="0.8 0.8 0.8 0.8"/>
+            </material>
         </visual>
         <collision>
@@ -190,6 +192,12 @@
     <joint name="lidar_joint" type="fixed">
         <parent link="base_link"/>
+        <child link="lidar_base"/>
+        <origin xyz="0.0 0.0 ${chassis_hight + lidar_width / 2}" rpy="0.0 0.0 0.0"/>
+    </joint>
+    <joint name="ldlidar_link_joint" type="fixed">
+        <parent link="lidar_base"/>
         <child link="lidar_frame"/>
-        <origin xyz="0.0 0.0 ${chassis_hight + lidar_width / 2}" rpy="0.0 0.0 0.0"/>
-    </joint>
+        <origin xyz="0 0 0.02745" rpy="0 0 0" />
+    </joint>
+    <link name="lidar_frame" />
 </robot>
